Commit message: Added grasping functionality. Can actually grasp a block. Block falls down though

File: me326_locobot_example/model/blue_cube.urdf (robot description, URDF)
Before this commit: robot blue_cube, 1 links, 0 joints
Links:
- link my_box: mass 0.5 -> 0.001

File: me326_locobot_example/model/green_cube.urdf (robot description, URDF)
Before this commit: robot green_cube, 1 links, 0 joints
Links:
- link my_box: mass 0.5 -> 0.001

File: me326_locobot_example/model/red_cube.urdf (robot description, URDF)
Before this commit: robot red_cube, 1 links, 0 joints
Links:
- link my_box: mass 0.5 -> 0.001

File: me326_locobot_example/model/yellow_cube.urdf (robot description, URDF)
Before this commit: robot yellow_cube, 1 links, 0 joints
Links:
- link my_box: mass 0.5 -> 0.001
